File: boostconverter.sch (KiCad schematic (older format))
At the start: 4 parts, among them Q9 BFS20W

Commit message: 2021-08-13
Parts:
- removed Q9: BFS20W, Package_TO_SOT_SMD:SOT-23, symbol Device:Q_NPN_BEC
- added C7: 10uF/2012, Capacitor_SMD:C_0805_2012Metric_Pad1.18x1.45mm_HandSolder, symbol Device:C
- added D4: SK24/SMB, Diode_SMD:D_SMB_Handsoldering, symbol Device:D_Schottky
- added Q8: BC846,215, Package_TO_SOT_SMD:SOT-23, symbol Device:Q_NPN_BEC
- L1: value 100uH -> 1mH; footprint Inductor_SMD:L_Vishay_IHLP-2020 -> inductor:SDR1307-102KL; MPN (none) -> SDR1307-102KL
- R17: value 2.7k -> 1k
Connections:
- net BATTERY: now also C6.1, L1.1; no longer L1.2
- net Earth: now also C7.2, Q8.2 (E)
- net HIGH_VOLTAGE: now also C7.1, D4.1 (K); no longer L1.1
- net SWITCH: now also R17.2; no longer C6.2, R17.1
- new net: Q8.1 (B), R17.1
- new net: C6.2, D4.2 (A), L1.2, Q8.3 (C)
Other:
- moved on the sheet: C6, L1, R17
Changed lines of the file:
@@
 Comment4 ""
 $EndDescr
-Text HLabel 4000 3000 0    50   Input ~ 0
+Text HLabel 6600 2350 2    50   Input ~ 0
 HIGH_VOLTAGE
 $Comp
 L Device:R R?
 U 1 1 6110B2A1
-P 5050 3350
+P 5150 2650
 AR Path="/610E7766/6110B2A1" Ref="R?"  Part="1"
 AR Path="/611083A4/6110B2A1" Ref="R17"  Part="1"
-F 0 "R17" V 5150 3300 50  0000 L CNN
-F 1 "2.7k" V 5050 3350 50  0000 C CNN
-F 2 "Resistor_SMD:R_0603_1608Metric_Pad0.98x0.95mm_HandSolder" V 4980 3350 50  0001 C CNN
-F 3 "~" H 5050 3350 50  0001 C CNN
-	1    5050 3350
+F 0 "R17" V 5250 2600 50  0000 L CNN
+F 1 "1k" V 5150 2650 50  0000 C CNN
+F 2 "Resistor_SMD:R_0603_1608Metric_Pad0.98x0.95mm_HandSolder" V 5080 2650 50  0001 C CNN
+F 3 "~" H 5150 2650 50  0001 C CNN
+	1    5150 2650
 	0    1    1    0
-$EndComp
-$Comp
-L Device:Q_NPN_BEC Q?
-U 1 1 6110B2A9
-P 4600 3350
-AR Path="/610E7766/6110B2A9" Ref="Q?"  Part="1"
-AR Path="/611083A4/6110B2A9" Ref="Q9"  Part="1"
-F 0 "Q9" H 4791 3396 50  0000 L CNN
-F 1 "BFS20W" H 4791 3305 50  0000 L CNN
-F 2 "Package_TO_SOT_SMD:SOT-23" H 4800 3450 50  0001 C CNN
-F 3 "~" H 4600 3350 50  0001 C CNN
-	1    4600 3350
-	-1   0    0    -1
 $EndComp
 $Comp
 L Device:L L1
 U 1 1 6111B5C3
-P 4650 2800
-F 0 "L1" V 4840 2800 50  0000 C CNN
-F 1 "100uH" V 4749 2800 50  0000 C CNN
-F 2 "Inductor_SMD:L_Vishay_IHLP-2020" H 4650 2800 50  0001 C CNN
-F 3 "~" H 4650 2800 50  0001 C CNN
-	1    4650 2800
+P 5350 2350
+F 0 "L1" V 5540 2350 50  0000 C CNN
+F 1 "1mH" V 5449 2350 50  0000 C CNN
+F 2 "inductor:SDR1307-102KL" H 5350 2350 50  0001 C CNN
+F 3 "https://www.digikey.kr/product-detail/ko/bourns-inc/SDR1307-102KL/SDR1307-102KLCT-ND/2352966" H 5350 2350 50  0001 C CNN
+F 4 "SDR1307-102KL" V 5350 2350 50  0001 C CNN "MPN"
+	1    5350 2350
 	0    -1   -1   0
 $EndComp
-Text HLabel 4900 2800 2    50   Input ~ 0
+Text HLabel 5200 2350 0    50   Input ~ 0
 BATTERY
-Wire Wire Line
-	4900 2800 4800 2800
-Wire Wire Line
-	4500 2800 4500 3000
-Wire Wire Line
-	4000 3000 4500 3000
-Connection ~ 4500 3000
-Wire Wire Line
-	4500 3000 4500 3150
-Wire Wire Line
-	4500 3550 4500 3750
-$Comp
-L power:Earth #PWR021
-U 1 1 6111D3A4
-P 4500 3750
-F 0 "#PWR021" H 4500 3500 50  0001 C CNN
-F 1 "Earth" H 4500 3600 50  0001 C CNN
-F 2 "" H 4500 3750 50  0001 C CNN
-F 3 "~" H 4500 3750 50  0001 C CNN
-	1    4500 3750
-	1    0    0    -1
-$EndComp
-Wire Wire Line
-	4800 3350 4850 3350
-Wire Wire Line
-	5200 3350 5250 3350
-Text HLabel 5300 3350 2    50   Input ~ 0
+Text HLabel 5000 2650 0    50   Input ~ 0
 SWITCH
 $Comp
 L Device:C C6
 U 1 1 6111E20B
-P 5050 3750
-F 0 "C6" V 4900 3750 50  0000 C CNN
-F 1 "10nF" V 5200 3750 50  0000 C CNN
-F 2 "Capacitor_SMD:C_0603_1608Metric_Pad1.08x0.95mm_HandSolder" H 5088 3600 50  0001 C CNN
-F 3 "~" H 5050 3750 50  0001 C CNN
-	1    5050 3750
+P 5350 1900
+F 0 "C6" V 5200 1900 50  0000 C CNN
+F 1 "10nF" V 5500 1900 50  0000 C CNN
+F 2 "Capacitor_SMD:C_0603_1608Metric_Pad1.08x0.95mm_HandSolder" H 5388 1750 50  0001 C CNN
+F 3 "~" H 5350 1900 50  0001 C CNN
+	1    5350 1900
 	0    -1   1    0
 $EndComp
+$Comp
+L Device:Q_NPN_BEC Q?
+U 1 1 61338A8D
+P 5500 2650
+AR Path="/610E7766/61338A8D" Ref="Q?"  Part="1"
+AR Path="/611083A4/61338A8D" Ref="Q8"  Part="1"
+F 0 "Q8" H 5690 2696 50  0000 L CNN
+F 1 "BC846,215" H 5690 2605 50  0000 L CNN
+F 2 "Package_TO_SOT_SMD:SOT-23" H 5700 2750 50  0001 C CNN
+F 3 "https://www.eleparts.co.kr/goods/view?no=4121178" H 5500 2650 50  0001 C CNN
+F 4 "BC846,215" H 5500 2650 50  0001 C CNN "MPN"
+	1    5500 2650
+	1    0    0    -1
+$EndComp
 Wire Wire Line
-	4900 3750 4850 3750
+	5600 2350 5600 2450
 Wire Wire Line
-	4850 3750 4850 3350
-Connection ~ 4850 3350
+	5500 2350 5600 2350
+$Comp
+L power:Earth #PWR022
+U 1 1 6133B061
+P 5600 2850
+F 0 "#PWR022" H 5600 2600 50  0001 C CNN
+F 1 "Earth" H 5600 2700 50  0001 C CNN
+F 2 "" H 5600 2850 50  0001 C CNN
+F 3 "~" H 5600 2850 50  0001 C CNN
+	1    5600 2850
+	1    0    0    -1
+$EndComp
 Wire Wire Line
-	4850 3350 4900 3350
+	5700 2350 5600 2350
+Connection ~ 5600 2350
 Wire Wire Line
-	5200 3750 5250 3750
+	5200 1900 5200 2350
 Wire Wire Line
-	5250 3750 5250 3350
-Connection ~ 5250 3350
+	5600 2350 5600 1900
 Wire Wire Line
-	5250 3350 5300 3350
+	5600 1900 5500 1900
+$Comp
+L Device:C C7
+U 1 1 6134A6D6
+P 6500 2600
+F 0 "C7" V 6350 2600 50  0000 C CNN
+F 1 "10uF/2012" V 6650 2600 50  0000 C CNN
+F 2 "Capacitor_SMD:C_0805_2012Metric_Pad1.18x1.45mm_HandSolder" H 6538 2450 50  0001 C CNN
+F 3 "~" H 6500 2600 50  0001 C CNN
+	1    6500 2600
+	-1   0    0    -1
+$EndComp
+$Comp
+L Device:D_Schottky D?
+U 1 1 6134D1A9
+P 5850 2350
+AR Path="/6134D1A9" Ref="D?"  Part="1"
+AR Path="/611083A4/6134D1A9" Ref="D4"  Part="1"
+F 0 "D4" H 5850 2133 50  0000 C CNN
+F 1 "SK24/SMB" H 5850 2224 50  0000 C CNN
+F 2 "Diode_SMD:D_SMB_Handsoldering" H 5850 2350 50  0001 C CNN
+F 3 "~" H 5850 2350 50  0001 C CNN
+F 4 "SK24" H 5850 2350 50  0001 C CNN "MPN"
+	1    5850 2350
+	-1   0    0    1
+$EndComp
+Wire Wire Line
+	6000 2350 6500 2350
+Wire Wire Line
+	6500 2450 6500 2350
+Connection ~ 6500 2350
+Wire Wire Line
+	6500 2350 6600 2350
+$Comp
+L power:Earth #PWR021
+U 1 1 6134E29E
+P 6500 2750
+F 0 "#PWR021" H 6500 2500 50  0001 C CNN
+F 1 "Earth" H 6500 2600 50  0001 C CNN
+F 2 "" H 6500 2750 50  0001 C CNN
+F 3 "~" H 6500 2750 50  0001 C CNN
+	1    6500 2750
+	1    0    0    -1
+$EndComp
 $EndSCHEMATC

Commit message: 2021-09-06
Parts:
- removed D4: SK24/SMB, Diode_SMD:D_SMB_Handsoldering, symbol Device:D_Schottky
- added D11: BAT54, Diode_SMD:D_SOT-23_ANK, symbol Diode:BAT54J
- C9: renamed from C7; value 10uF/2012 -> 10uF/3225; footprint Capacitor_SMD:C_0805_2012Metric_Pad1.18x1.45mm_HandSolder -> Capacitor_SMD:C_1210_3225Metric; MPN (none) -> UMK325BJ106MM-P
- L1: footprint inductor:SDR1307-102KL -> Inductor_SMD:L_Bourns-SRN4018; MPN SDR1307-102KL -> SC4532D-102K
- renumbered C6 to C8, R17 to R25
Connections:
- net HIGH_VOLTAGE: now also D11.1 (K)
- net at C8.2, L1.2, Q8.3 (C): now also D11.2 (A)
Changed lines of the file:
@@
 P 5150 2650
 AR Path="/610E7766/6110B2A1" Ref="R?"  Part="1"
-AR Path="/611083A4/6110B2A1" Ref="R17"  Part="1"
-F 0 "R17" V 5250 2600 50  0000 L CNN
+AR Path="/611083A4/6110B2A1" Ref="R25"  Part="1"
+F 0 "R25" V 5250 2600 50  0000 L CNN
 F 1 "1k" V 5150 2650 50  0000 C CNN
 F 2 "Resistor_SMD:R_0603_1608Metric_Pad0.98x0.95mm_HandSolder" V 5080 2650 50  0001 C CNN
@@
 F 0 "L1" V 5540 2350 50  0000 C CNN
 F 1 "1mH" V 5449 2350 50  0000 C CNN
-F 2 "inductor:SDR1307-102KL" H 5350 2350 50  0001 C CNN
-F 3 "https://www.digikey.kr/product-detail/ko/bourns-inc/SDR1307-102KL/SDR1307-102KLCT-ND/2352966" H 5350 2350 50  0001 C CNN
-F 4 "SDR1307-102KL" V 5350 2350 50  0001 C CNN "MPN"
+F 2 "Inductor_SMD:L_Bourns-SRN4018" H 5350 2350 50  0001 C CNN
+F 3 "https://www.ic114.com/WebSite/site/sc/00V0.aspx?id_p=P0083538" H 5350 2350 50  0001 C CNN
+F 4 "SC4532D-102K" V 5350 2350 50  0001 C CNN "MPN"
 	1    5350 2350
 	0    -1   -1   0
@@
 SWITCH
 $Comp
-L Device:C C6
+L Device:C C8
 U 1 1 6111E20B
 P 5350 1900
-F 0 "C6" V 5200 1900 50  0000 C CNN
+F 0 "C8" V 5200 1900 50  0000 C CNN
 F 1 "10nF" V 5500 1900 50  0000 C CNN
 F 2 "Capacitor_SMD:C_0603_1608Metric_Pad1.08x0.95mm_HandSolder" H 5388 1750 50  0001 C CNN
@@
 	5500 2350 5600 2350
 $Comp
-L power:Earth #PWR022
+L power:Earth #PWR023
 U 1 1 6133B061
 P 5600 2850
-F 0 "#PWR022" H 5600 2600 50  0001 C CNN
+F 0 "#PWR023" H 5600 2600 50  0001 C CNN
 F 1 "Earth" H 5600 2700 50  0001 C CNN
 F 2 "" H 5600 2850 50  0001 C CNN
@@
 	5600 1900 5500 1900
 $Comp
-L Device:C C7
+L Device:C C9
 U 1 1 6134A6D6
 P 6500 2600
-F 0 "C7" V 6350 2600 50  0000 C CNN
-F 1 "10uF/2012" V 6650 2600 50  0000 C CNN
-F 2 "Capacitor_SMD:C_0805_2012Metric_Pad1.18x1.45mm_HandSolder" H 6538 2450 50  0001 C CNN
-F 3 "~" H 6500 2600 50  0001 C CNN
+F 0 "C9" V 6350 2600 50  0000 C CNN
+F 1 "10uF/3225" V 6650 2600 50  0000 C CNN
+F 2 "Capacitor_SMD:C_1210_3225Metric" H 6538 2450 50  0001 C CNN
+F 3 "https://www.eleparts.co.kr/goods/view?no=10504698" H 6500 2600 50  0001 C CNN
+F 4 "UMK325BJ106MM-P" V 6500 2600 50  0001 C CNN "MPN"
 	1    6500 2600
 	-1   0    0    -1
-$EndComp
-$Comp
-L Device:D_Schottky D?
-U 1 1 6134D1A9
-P 5850 2350
-AR Path="/6134D1A9" Ref="D?"  Part="1"
-AR Path="/611083A4/6134D1A9" Ref="D4"  Part="1"
-F 0 "D4" H 5850 2133 50  0000 C CNN
-F 1 "SK24/SMB" H 5850 2224 50  0000 C CNN
-F 2 "Diode_SMD:D_SMB_Handsoldering" H 5850 2350 50  0001 C CNN
-F 3 "~" H 5850 2350 50  0001 C CNN
-F 4 "SK24" H 5850 2350 50  0001 C CNN "MPN"
-	1    5850 2350
-	-1   0    0    1
 $EndComp
 Wire Wire Line
@@
 	6500 2350 6600 2350
 $Comp
-L power:Earth #PWR021
+L power:Earth #PWR022
 U 1 1 6134E29E
 P 6500 2750
-F 0 "#PWR021" H 6500 2500 50  0001 C CNN
+F 0 "#PWR022" H 6500 2500 50  0001 C CNN
 F 1 "Earth" H 6500 2600 50  0001 C CNN
 F 2 "" H 6500 2750 50  0001 C CNN
@@
 	1    0    0    -1
 $EndComp
+$Comp
+L Diode:BAT54J D?
+U 1 1 613AAFF8
+P 5850 2350
+AR Path="/613AAFF8" Ref="D?"  Part="1"
+AR Path="/611083A4/613AAFF8" Ref="D11"  Part="1"
+F 0 "D11" H 5850 2567 50  0000 C CNN
+F 1 "BAT54" H 5850 2476 50  0000 C CNN
+F 2 "Diode_SMD:D_SOT-23_ANK" H 5850 2175 50  0001 C CNN
+F 3 "https://www.eleparts.co.kr/goods/view?no=6531921" H 5850 2350 50  0001 C CNN
+F 4 "BAT54" V 5850 2350 50  0001 C CNN "MPN"
+	1    5850 2350
+	-1   0    0    -1
+$EndComp
 $EndSCHEMATC
