File: h-bridge.sch (KiCad schematic (older format))
At the start: 16 parts, among them Q2 MMBT5401, Q3 MMBT5401, Q4 MMBT5401, Q5 MMBT5401, Q6 MMBT5401, Q7 BFS20W, Q8 BFS20W

Commit message: 2021-08-13
Parts:
- removed Q6: MMBT5401, Package_TO_SOT_SMD:SOT-23, symbol Device:Q_PNP_BEC
- removed Q8: BFS20W, Package_TO_SOT_SMD:SOT-23, symbol Device:Q_NPN_BEC
- added Q6: BC846,215, Package_TO_SOT_SMD:SOT-23, symbol Device:Q_NPN_BEC
- Q2, Q3, Q4, Q5: value MMBT5401 -> BC856B,215; MPN (none) -> BC856B,215
- Q7: value BFS20W -> BC846,215; MPN (none) -> BC846,215
- R8: value 100 -> 0
- renumbered R15 to R14, R14 to R15
Connections:
- net BATTERY is gone; now on net HIGH_VOLTAGE: R8.1
- net Earth: now also Q6.2 (E)
- net OUTH: now also Q2.3 (C), Q4.2 (E); no longer Q2.2 (E), Q4.3 (C)
- net OUTL: now also Q3.3 (C), Q5.2 (E); no longer Q3.2 (E), Q5.3 (C)
- net SENS: now also Q2.2 (E), Q3.2 (E); no longer Q2.3 (C), Q3.3 (C)
- net at R15.1: now also Q6.1 (B); no longer Q7.1 (B)
- net at R12.2, R13.1, R9.2: now also Q6.3 (C); no longer Q7.3 (C)
- net at R13.2, R14.2: now also Q4.3 (C), Q5.3 (C); no longer Q4.2 (E), Q5.2 (E)
- net at R10.2, R11.2, R14.1: now also Q7.3 (C)
- net at R16.1: now also Q7.1 (B)
Other:
- moved on the sheet: R14, R16
Changed lines of the file:
@@
 Comment4 ""
 $EndDescr
-Text HLabel 3900 1500 0    50   Input ~ 0
-BATTERY
 $Comp
 L Device:R R8
@@
 P 4000 1750
 F 0 "R8" V 4100 1700 50  0000 L CNN
-F 1 "100" V 4000 1750 50  0000 C CNN
+F 1 "0" V 4000 1750 50  0000 C CNN
 F 2 "Resistor_SMD:R_0603_1608Metric_Pad0.98x0.95mm_HandSolder" V 3930 1750 50  0001 C CNN
 F 3 "~" H 4000 1750 50  0001 C CNN
@@
 Wire Wire Line
 	4000 1500 4000 1600
-$Comp
-L Device:Q_PNP_BEC Q2
-U 1 1 610F0C17
-P 2900 2300
-F 0 "Q2" H 3091 2346 50  0000 L CNN
-F 1 "MMBT5401" H 3091 2255 50  0000 L CNN
-F 2 "Package_TO_SOT_SMD:SOT-23" H 3100 2400 50  0001 C CNN
-F 3 "~" H 2900 2300 50  0001 C CNN
-	1    2900 2300
-	1    0    0    -1
-$EndComp
-$Comp
-L Device:Q_NPN_BEC Q7
-U 1 1 610F1FB4
-P 2900 4400
-F 0 "Q7" H 3091 4446 50  0000 L CNN
-F 1 "BFS20W" H 3091 4355 50  0000 L CNN
-F 2 "Package_TO_SOT_SMD:SOT-23" H 3100 4500 50  0001 C CNN
-F 3 "~" H 2900 4400 50  0001 C CNN
-	1    2900 4400
-	1    0    0    -1
-$EndComp
-$Comp
-L Device:Q_PNP_BEC Q3
-U 1 1 610F363F
-P 5100 2300
-F 0 "Q3" H 5291 2346 50  0000 L CNN
-F 1 "MMBT5401" H 5291 2255 50  0000 L CNN
-F 2 "Package_TO_SOT_SMD:SOT-23" H 5300 2400 50  0001 C CNN
-F 3 "~" H 5100 2300 50  0001 C CNN
-	1    5100 2300
-	-1   0    0    -1
-$EndComp
-$Comp
-L Device:Q_PNP_BEC Q4
-U 1 1 610F5EF2
-P 2900 3200
-F 0 "Q4" H 3091 3246 50  0000 L CNN
-F 1 "MMBT5401" H 3091 3155 50  0000 L CNN
-F 2 "Package_TO_SOT_SMD:SOT-23" H 3100 3300 50  0001 C CNN
-F 3 "~" H 2900 3200 50  0001 C CNN
-	1    2900 3200
-	1    0    0    -1
-$EndComp
-$Comp
-L Device:Q_PNP_BEC Q5
-U 1 1 610F6D0C
-P 5100 3200
-F 0 "Q5" H 5291 3246 50  0000 L CNN
-F 1 "MMBT5401" H 5291 3155 50  0000 L CNN
-F 2 "Package_TO_SOT_SMD:SOT-23" H 5300 3300 50  0001 C CNN
-F 3 "~" H 5100 3200 50  0001 C CNN
-	1    5100 3200
-	-1   0    0    -1
-$EndComp
 $Comp
 L Device:R R9
@@
 Connection ~ 3000 3500
 $Comp
+L Device:R R14
+U 1 1 610FB38E
+P 5000 3850
+F 0 "R14" V 5100 3800 50  0000 L CNN
+F 1 "33k" V 5000 3850 50  0000 C CNN
+F 2 "Resistor_SMD:R_0603_1608Metric_Pad0.98x0.95mm_HandSolder" V 4930 3850 50  0001 C CNN
+F 3 "~" H 5000 3850 50  0001 C CNN
+	1    5000 3850
+	-1   0    0    1
+$EndComp
+Wire Wire Line
+	3000 4200 3000 4100
+$Comp
 L Device:R R15
-U 1 1 610FB38E
-P 5300 4450
-F 0 "R15" V 5400 4400 50  0000 L CNN
-F 1 "33k" V 5300 4450 50  0000 C CNN
-F 2 "Resistor_SMD:R_0603_1608Metric_Pad0.98x0.95mm_HandSolder" V 5230 4450 50  0001 C CNN
-F 3 "~" H 5300 4450 50  0001 C CNN
-	1    5300 4450
-	-1   0    0    1
-$EndComp
-Connection ~ 5000 3500
-Wire Wire Line
-	3000 4200 3000 4100
-$Comp
-L Device:Q_NPN_BEC Q8
-U 1 1 610FCD91
-P 5400 4900
-F 0 "Q8" H 5591 4946 50  0000 L CNN
-F 1 "BFS20W" H 5591 4855 50  0000 L CNN
-F 2 "Package_TO_SOT_SMD:SOT-23" H 5600 5000 50  0001 C CNN
-F 3 "~" H 5400 4900 50  0001 C CNN
-	1    5400 4900
-	-1   0    0    -1
-$EndComp
-Wire Wire Line
-	5300 4700 5300 4650
-$Comp
-L Device:R R14
 U 1 1 610FE429
 P 2450 4400
-F 0 "R14" V 2550 4350 50  0000 L CNN
+F 0 "R15" V 2550 4350 50  0000 L CNN
 F 1 "1k" V 2450 4400 50  0000 C CNN
 F 2 "Resistor_SMD:R_0603_1608Metric_Pad0.98x0.95mm_HandSolder" V 2380 4400 50  0001 C CNN
@@
 L Device:R R16
 U 1 1 610FECA5
-P 5850 4900
-F 0 "R16" V 5950 4850 50  0000 L CNN
-F 1 "1k" V 5850 4900 50  0000 C CNN
-F 2 "Resistor_SMD:R_0603_1608Metric_Pad0.98x0.95mm_HandSolder" V 5780 4900 50  0001 C CNN
-F 3 "~" H 5850 4900 50  0001 C CNN
-	1    5850 4900
+P 5550 4400
+F 0 "R16" V 5650 4350 50  0000 L CNN
+F 1 "1k" V 5550 4400 50  0000 C CNN
+F 2 "Resistor_SMD:R_0603_1608Metric_Pad0.98x0.95mm_HandSolder" V 5480 4400 50  0001 C CNN
+F 3 "~" H 5550 4400 50  0001 C CNN
+	1    5550 4400
 	0    -1   -1   0
 $EndComp
 Wire Wire Line
-	5700 4900 5600 4900
+	5400 4400 5300 4400
 $Comp
 L power:Earth #PWR019
@@
 L power:Earth #PWR020
 U 1 1 610FFBAA
-P 5300 5100
-F 0 "#PWR020" H 5300 4850 50  0001 C CNN
-F 1 "Earth" H 5300 4950 50  0001 C CNN
-F 2 "" H 5300 5100 50  0001 C CNN
-F 3 "~" H 5300 5100 50  0001 C CNN
-	1    5300 5100
+P 5000 4600
+F 0 "#PWR020" H 5000 4350 50  0001 C CNN
+F 1 "Earth" H 5000 4450 50  0001 C CNN
+F 2 "" H 5000 4600 50  0001 C CNN
+F 3 "~" H 5000 4600 50  0001 C CNN
+	1    5000 4600
 	1    0    0    -1
 $EndComp
@@
 Text HLabel 2300 4400 0    50   Input ~ 0
 SW_POS
-Text HLabel 6000 4900 2    50   Input ~ 0
+Text HLabel 5700 4400 2    50   Input ~ 0
 SW_NEG
 Text HLabel 2900 2000 0    50   Input ~ 0
@@
 	2900 2000 3000 2000
 Connection ~ 3000 2000
-Text HLabel 6000 3700 2    50   Input ~ 0
+Text HLabel 3900 1500 0    50   Input ~ 0
 HIGH_VOLTAGE
-$Comp
-L Device:Q_PNP_BEC Q6
-U 1 1 6110DA48
-P 5200 4000
-F 0 "Q6" H 5391 4046 50  0000 L CNN
-F 1 "MMBT5401" H 5391 3955 50  0000 L CNN
-F 2 "Package_TO_SOT_SMD:SOT-23" H 5400 4100 50  0001 C CNN
-F 3 "~" H 5200 4000 50  0001 C CNN
-	1    5200 4000
+Wire Wire Line
+	5900 2300 5900 4100
+$Comp
+L Device:Q_PNP_BEC Q3
+U 1 1 61334FF6
+P 5100 2300
+F 0 "Q3" H 5291 2254 50  0000 L CNN
+F 1 "BC856B,215" H 5291 2345 50  0000 L CNN
+F 2 "Package_TO_SOT_SMD:SOT-23" H 5300 2400 50  0001 C CNN
+F 3 "https://www.eleparts.co.kr/goods/view?no=72756" H 5100 2300 50  0001 C CNN
+F 4 "BC856B,215" H 5100 2300 50  0001 C CNN "MPN"
+	1    5100 2300
+	-1   0    0    1
+$EndComp
+$Comp
+L Device:Q_NPN_BEC Q6
+U 1 1 61335335
+P 2900 4400
+F 0 "Q6" H 3090 4446 50  0000 L CNN
+F 1 "BC846,215" H 3090 4355 50  0000 L CNN
+F 2 "Package_TO_SOT_SMD:SOT-23" H 3100 4500 50  0001 C CNN
+F 3 "https://www.eleparts.co.kr/goods/view?no=4121178" H 2900 4400 50  0001 C CNN
+F 4 "BC846,215" H 2900 4400 50  0001 C CNN "MPN"
+	1    2900 4400
 	1    0    0    -1
 $EndComp
-Wire Wire Line
-	5000 3500 5000 4000
-Wire Wire Line
-	5300 4200 5000 4200
-Wire Wire Line
-	5000 4200 5000 4000
-Connection ~ 5000 4000
-Wire Wire Line
-	5300 4300 5300 4200
-Connection ~ 5300 4200
-Wire Wire Line
-	5300 4650 5900 4650
-Wire Wire Line
-	5900 2300 5900 4650
-Connection ~ 5300 4650
-Wire Wire Line
-	5300 4650 5300 4600
-Wire Wire Line
-	6000 3700 5300 3700
-Wire Wire Line
-	5300 3700 5300 3800
+$Comp
+L Device:Q_PNP_BEC Q5
+U 1 1 61340240
+P 5100 3200
+F 0 "Q5" H 5291 3154 50  0000 L CNN
+F 1 "BC856B,215" H 5291 3245 50  0000 L CNN
+F 2 "Package_TO_SOT_SMD:SOT-23" H 5300 3300 50  0001 C CNN
+F 3 "https://www.eleparts.co.kr/goods/view?no=72756" H 5100 3200 50  0001 C CNN
+F 4 "BC856B,215" H 5100 3200 50  0001 C CNN "MPN"
+	1    5100 3200
+	-1   0    0    1
+$EndComp
+$Comp
+L Device:Q_PNP_BEC Q2
+U 1 1 61340D3F
+P 2900 2300
+F 0 "Q2" H 3090 2254 50  0000 L CNN
+F 1 "BC856B,215" H 3090 2345 50  0000 L CNN
+F 2 "Package_TO_SOT_SMD:SOT-23" H 3100 2400 50  0001 C CNN
+F 3 "https://www.eleparts.co.kr/goods/view?no=72756" H 2900 2300 50  0001 C CNN
+F 4 "BC856B,215" H 2900 2300 50  0001 C CNN "MPN"
+	1    2900 2300
+	1    0    0    1
+$EndComp
+$Comp
+L Device:Q_PNP_BEC Q4
+U 1 1 6134203D
+P 2900 3200
+F 0 "Q4" H 3090 3154 50  0000 L CNN
+F 1 "BC856B,215" H 3090 3245 50  0000 L CNN
+F 2 "Package_TO_SOT_SMD:SOT-23" H 3100 3300 50  0001 C CNN
+F 3 "https://www.eleparts.co.kr/goods/view?no=72756" H 2900 3200 50  0001 C CNN
+F 4 "BC856B,215" H 2900 3200 50  0001 C CNN "MPN"
+	1    2900 3200
+	1    0    0    1
+$EndComp
+Wire Wire Line
+	5000 3700 5000 3500
+Connection ~ 5000 3500
+$Comp
+L Device:Q_NPN_BEC Q7
+U 1 1 61345621
+P 5100 4400
+F 0 "Q7" H 5291 4446 50  0000 L CNN
+F 1 "BC846,215" H 5291 4355 50  0000 L CNN
+F 2 "Package_TO_SOT_SMD:SOT-23" H 5300 4500 50  0001 C CNN
+F 3 "https://www.eleparts.co.kr/goods/view?no=4121178" H 5100 4400 50  0001 C CNN
+F 4 "BC846,215" H 5100 4400 50  0001 C CNN "MPN"
+	1    5100 4400
+	-1   0    0    -1
+$EndComp
+Wire Wire Line
+	5000 4200 5000 4100
+Wire Wire Line
+	5000 4100 5900 4100
+Connection ~ 5000 4100
+Wire Wire Line
+	5000 4100 5000 4000
 $EndSCHEMATC

Commit message: 2021-09-06
Parts:
- removed R8: 0, Resistor_SMD:R_0603_1608Metric_Pad0.98x0.95mm_HandSolder, symbol Device:R
- added D10: Zenor/3.3V, Diode_SMD:D_MiniMELF, symbol Diode:ZMMxx
- added D9: Zenor/47V, Diode_SMD:D_MiniMELF, symbol Diode:ZMMxx
- added R13: 1M, Resistor_SMD:R_0603_1608Metric_Pad0.98x0.95mm_HandSolder, symbol Device:R
- added R14, R16: 33k, Resistor_SMD:R_0603_1608Metric_Pad0.98x0.95mm_HandSolder, symbol Device:R
- added R15: 100k, Resistor_SMD:R_0603_1608Metric_Pad0.98x0.95mm_HandSolder, symbol Device:R
- R22: renamed from R14; value 33k -> 0
- R23: renamed from R15; value 1k -> 100
- R24: renamed from R16; value 1k -> 100
- renumbered R9 to R17, R10 to R18, R11 to R19, R12 to R20, R13 to R21
Connections:
- net Earth: now also D10.2 (A), R15.1
- net HIGH_VOLTAGE: now also Q2.2 (E), Q3.2 (E), D9.1 (K), R14.1, R16.1
- net SENS: now also D10.1 (K), R13.1, R15.2; no longer Q2.2 (E), Q3.2 (E)
- net at Q6.3 (C), R17.2, R20.2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: now also R14.2
- net at Q7.3 (C), R18.2, R19.2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: now also R16.2
- new net: D9.2 (A), R13.2
Other:
- moved on the sheet: Q2, Q3, Q4, Q5, Q6, Q7, R17, R18, R19, R20, R21, R22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
