File: lfmassage.sch (KiCad schematic (older format))
At the start: 26 parts, among them J1 Batt, J2 OUT, J3 ESP_DEVKITC, Q1 BFS20W, SW1 NW3-A03-05, SW2 SW_Push, SW3 SW_Push, SW4 SW_Push, U1 USB_CType_6Pin, U2 MCP73831

Commit message: 2021-08-13
Parts:
- D1, D3: value SK24/SMA -> SK24/SMB; footprint Diode_SMD:D_SMA_Handsoldering -> Diode_SMD:D_SMB_Handsoldering
- R2: value 2k -> 10k
Changed lines of the file:
@@
 P 3650 1050
 F 0 "D1" H 3650 833 50  0000 C CNN
-F 1 "SK24/SMA" H 3650 924 50  0000 C CNN
-F 2 "Diode_SMD:D_SMA_Handsoldering" H 3650 1050 50  0001 C CNN
+F 1 "SK24/SMB" H 3650 924 50  0000 C CNN
+F 2 "Diode_SMD:D_SMB_Handsoldering" H 3650 1050 50  0001 C CNN
 F 3 "~" H 3650 1050 50  0001 C CNN
 F 4 "SK24" H 3650 1050 50  0001 C CNN "MPN"
@@
 P 3400 1900
 F 0 "R2" V 3300 1950 50  0000 R CNN
-F 1 "2k" V 3400 1900 50  0000 C CNN
+F 1 "10k" V 3400 1900 50  0000 C CNN
 F 2 "Resistor_SMD:R_0603_1608Metric_Pad0.98x0.95mm_HandSolder" V 3330 1900 50  0001 C CNN
 F 3 "~" H 3400 1900 50  0001 C CNN
@@
 F0 "H-Bridge" 50
 F1 "h-bridge.sch" 50
-F2 "BATTERY" I L 7950 1300 50
-F3 "OUTH" I R 9400 1750 50
-F4 "OUTL" I R 9400 2050 50
-F5 "SW_POS" I L 7950 2350 50
-F6 "SW_NEG" I L 7950 2500 50
-F7 "SENS" I L 7950 2200 50
-F8 "HIGH_VOLTAGE" I L 7950 1400 50
+F2 "OUTH" I R 9400 1750 50
+F3 "OUTL" I R 9400 2050 50
+F4 "SW_POS" I L 7950 2350 50
+F5 "SW_NEG" I L 7950 2500 50
+F6 "SENS" I L 7950 2200 50
+F7 "HIGH_VOLTAGE" I L 7950 1400 50
 $EndSheet
 $Sheet
@@
 Wire Wire Line
 	7700 1400 7950 1400
-Text GLabel 7950 1300 0    50   Input ~ 0
-BATT
 $Comp
 L Switch:SW_Push SW1
@@
 P 3900 6350
 F 0 "D3" H 3950 6450 50  0000 L CNN
-F 1 "SK24/SMA" H 3750 6250 50  0000 L CNN
-F 2 "Diode_SMD:D_SMA_Handsoldering" H 3900 6350 50  0001 C CNN
+F 1 "SK24/SMB" H 3750 6250 50  0000 L CNN
+F 2 "Diode_SMD:D_SMB_Handsoldering" H 3900 6350 50  0001 C CNN
 F 3 "~" H 3900 6350 50  0001 C CNN
 F 4 "SK24" H 3900 6350 50  0001 C CNN "MPN"

Commit message: 2021-09-06
Parts:
- removed C5: 100nF/1608, Capacitor_SMD:C_0603_1608Metric_Pad1.08x0.95mm_HandSolder, symbol Device:C
- removed D1, D3: SK24/SMB, Diode_SMD:D_SMB_Handsoldering, symbol Device:D_Schottky
- removed J3: ESP_DEVKITC, espressif:ESP32_DEVKITC, symbol Connector_Generic:Conn_02x15_Counter_Clockwise
- removed SW2, SW3, SW4: SW_Push, ali_Switch:NW3-A03-05, symbol Switch:SW_Push
- added C2, C4: 100nF/1608, Capacitor_SMD:C_0603_1608Metric_Pad1.08x0.95mm_HandSolder, symbol Device:C
- added C3: 10nF/1608, Capacitor_SMD:C_0603_1608Metric_Pad1.08x0.95mm_HandSolder, symbol Device:C
- added D2: BAT54, Diode_SMD:D_SOT-23_ANK, symbol Diode:BAT54J
- added D3: RED, LED_SMD:LED_0603_1608Metric, symbol Device:LED
- added D4: BLU, LED_SMD:LED_0603_1608Metric, symbol Device:LED
- added D5: WHT, LED_SMD:LED_0603_1608Metric, symbol Device:LED
- added D6, D8: RED, LED_SMD:LED_1206_3216Metric, symbol Device:LED
- added D7: IR, LED_SMD:LED_1206_3216Metric, symbol Device:LED
- added J3: ISP, Connector_PinHeader_2.54mm:PinHeader_1x03_P2.54mm_Vertical, symbol Connector_Generic:Conn_01x03
- added K2: +, Button_Switch_SMD:SW_SPST_B3SL-1002P, symbol Switch:SW_Push
- added K3: -, Button_Switch_SMD:SW_SPST_B3SL-1002P, symbol Switch:SW_Push
- added R10, R8: 220, Resistor_SMD:R_0603_1608Metric_Pad0.98x0.95mm_HandSolder, symbol Device:R
- added R5, R7: 560, Resistor_SMD:R_0603_1608Metric_Pad0.98x0.95mm_HandSolder, symbol Device:R
- added R9: 100, Resistor_SMD:R_0603_1608Metric_Pad0.98x0.95mm_HandSolder, symbol Device:R
- added U3: MIC5318-2.8YD5-TR, Package_TO_SOT_SMD:TSOT-23-5, symbol MIC531833YD5TR:MIC5318-3.3YD5-TR
- added U4: EFM8BB10F8G-A-SOIC16, Package_SO:SOIC-16_3.9x9.9mm_P1.27mm, symbol MCU_SiliconLabs:EFM8BB10F8G-A-SOIC16
- BZ1: value IMT09B2703P -> BST-5533S; footprint Buzzer_Beeper:MagneticBuzzer_PUI_AT-0927-TT-6-R -> buzzer:BST-5533S; MPN (none) -> BST-5533S
- K1: renamed from SW1; value NW3-A03-05 -> MODE; footprint ali_Switch:NW3-A03-05 -> Button_Switch_SMD:SW_SPST_B3SL-1002P; MPN (none) -> PTS526
- Q1: value BFS20W -> S8050
- R3: renamed from R7; value 100 -> 150
- R6: value 1k -> 560
- renumbered C2 to C5, C3 to C6, C4 to C7, D2 to D1, R4 to R11, R5 to R12, R3 to R4
Connections:
- net D25 is gone; now on net VCC: R12.2
- net D26 is gone; now on net VCC: R11.2
- net D27 is gone; now on net VCC: R4.2
- net BATT: now also C2.1, U3.1 (IN), U3.3 (EN)
- net Earth: now also K1.1, C2.2, C3.2, C4.2, J3.1 (Pin_1), K2.1, K3.1, U3.2 (GND), U4.4 (GND)
- net VBUS: now also D1.2 (A), U2.4 (VDD)
- net P0.0(MODE): now reaches C5.1, K1.2, R4.1
- net P0.0(MODE): now also U4.3 (P0.0)
- net P0.1(+): now reaches C6.1, R11.1
- net P0.1(+): now also K2.2, U4.2 (P0.1)
- net P0.2(-): now reaches C7.1, R12.1
- net P0.2(-): now also K3.2, U4.1 (P0.2)
- net VCC: now reaches R6.1
- net VCC: now also BZ1.1 (-), C4.1, D2.1 (K), R10.1, R5.1, R7.1, R8.1, R9.1, U3.5 (OUT), U4.5 (VDD)
- net at BZ1.2 (+), Q1.3 (C): now also D2.2 (A)
- removed net +3V3: BZ1.1 (-), K1.1
- net D22 renamed P0.7(BUZZER)
- net P0.7(BUZZER): now also U4.12 (P0.7)
- net D33: no longer names the net of R6.2
- net D33: now also D4.2 (A)
- new net: C3.1, U3.4 (BYP)
- new net: D6.2 (A), R8.2
- new net: D7.2 (A), R9.2
- new net: D8.2 (A), R10.2
- new net: D3.2 (A), R5.2
- new net: D5.2 (A), R7.2
- new net C2CK: J3.2 (Pin_2), U4.6 (RSTb/C2CK)
- new net C2D: J3.3 (Pin_3), U4.7 (P2.0/C2D)
- new net P0.3(RED): D3.1 (K), U4.16 (P0.3)
- new net P0.4(BLU): D4.1 (K), U4.15 (P0.4)
- new net P0.5(WHT): D5.1 (K), U4.14 (P0.5)
- new net P0.6(IRLED): D6.1 (K), D7.1 (K), D8.1 (K), U4.13 (P0.6)
- new net P1.0(SW): U4.11 (P1.0)
- new net P1.1(POS): U4.10 (P1.1)
- new net P1.2(NEG): U4.9 (P1.2)
- new net P1.3(SENS): U4.8 (P1.3)
- no-connect marks 4 -> 0
Other:
- moved on the sheet: BZ1, C1, C5, C6, C7, D1, J1, K1, Q1, R1, R11, R12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

Commit message: 2021-09-26
Parts:
- added C10: 10uF/1608, Capacitor_SMD:C_0603_1608Metric_Pad1.08x0.95mm_HandSolder, symbol Device:C
- C1: value 10uF/2012 -> 10uF/1608; footprint Capacitor_SMD:C_0805_2012Metric_Pad1.18x1.45mm_HandSolder -> Capacitor_SMD:C_0603_1608Metric
- D1: value LED/2012 -> LED/1608; footprint LED_SMD:LED_0805_2012Metric_Pad1.15x1.40mm_HandSolder -> LED_SMD:LED_0603_1608Metric
- D3: value RED -> LED/1608
- D4: value BLU -> LED/1608
- D5: value WHT -> LED/1608
- J1: footprint Connector_Molex:Molex_PicoBlade_53261-0271_1x02-1MP_P1.25mm_Horizontal -> Connector_Molex:Molex_PicoBlade_53398-0271_1x02-1MP_P1.25mm_Vertical
- J2: value OUT -> electrode; footprint Connector_PinHeader_2.54mm:PinHeader_1x02_P2.54mm_Vertical -> lfmassage_pad:electrode
- K1, K2, K3: footprint Button_Switch_SMD:SW_SPST_B3SL-1002P -> Button_Switch_SMD:Panasonic_EVQPUJ_EVQPUA; MPN PTS526 -> EVQ-P7A01P
Connections:
- net Earth: now also C10.2
- net H-Bridge/OUTH: now also J2.2 (Pin_2); no longer J2.1 (Pin_1)
- net H-Bridge/OUTL: now also J2.1 (Pin_1); no longer J2.2 (Pin_2)
- net P0.3(RED): now also R5.2; no longer D3.1 (K)
- net VCC: now also D3.2 (A), D4.2 (A), D5.2 (A), C10.1; no longer R5.1, R6.1, R7.1
- net P0.4(GRN): now reaches R6.2
- net P0.4(GRN): now also U4.15 (P0.4); no longer D4.2 (A)
- net P0.5(BLU): now reaches R7.2
- net P0.5(BLU): now also U4.14 (P0.5); no longer D5.2 (A)
- net P0.0(MODE) renamed P0.1(MODE)
- net P0.1(MODE): now also U4.2 (P0.1); no longer U4.3 (P0.0)
- net P0.1(+) renamed P0.0(+)
- net P0.0(+): now also U4.3 (P0.0); no longer U4.2 (P0.1)
- net P0.4(BLU): no longer names the net of D4.1 (K)
- net P0.4(BLU): now also R6.1; no longer U4.15 (P0.4)
- net P0.5(WHT): no longer names the net of D5.1 (K)
- net P0.5(WHT): now also R7.1; no longer U4.14 (P0.5)
- net P1.0(SW) renamed P1.0(NEG)
- net P1.2(NEG) renamed P1.2(SW)
- new net: D3.1 (K), R5.1
Other:
- moved on the sheet: R5, R6, R7
